File: Kicad arduino uno/Capteur_graphite/Capteur_graphite.kicad_pcb (KiCad board)
At the start: 2 copper layers, 68.6 x 53.3 mm, 25 parts, among them J1 Power, J2 Digital/PWM, J3 Analog, J4 Digital/PWM, U3 MCP41050, U4 LTC1050

Commit message: pcb_verifiée_prêt_à_percer
Parts:
- moved C1 9.00 mm to (111.0, 60.5)
- moved C4 7.00 mm to (125.5, 88.0)
- moved R3 7.00 mm to (120.0, 82.0)
- moved U5 6.00 mm to (106.5, 79.5)
Routing:
- net Net-(U3-PB0): track 39.7 -> 28.3 mm
- net Net-(C4-Pad1): track 24.4 -> 17.4 mm
- net Net-(U5-OUT): track 4.00 -> 7.66 mm
- net +5V: track 176.6 -> 173.7 mm
Changed lines of the file:
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@@
 		(grid_origin 100 100)
 		(pcbplotparams
-			(layerselection 0x0000030_80000001)
+			(layerselection 0x0000000_fffffffe)
 			(plot_on_all_layers_selection 0x0000000_00000000)
 			(disableapertmacros no)
@@
 			(sketchpadsonfab no)
 			(subtractmaskfromsilk no)
-			(outputformat 1)
+			(outputformat 4)
 			(mirror no)
-			(drillshape 1)
+			(drillshape 0)
 			(scaleselection 1)
-			(outputdirectory "")
+			(outputdirectory "../Gerber/")
 		)
 	)
@@
 	(footprint "Librairie_d_empreinte:Capteur"
 		(layer "F.Cu")
-		(at 106.5 73.5)
+		(at 106.5 79.5)
 		(property "Reference" "U5"
 			(at 0 -0.5 0)
@@
 	(footprint "Capacitor_THT:C_Disc_D7.0mm_W2.5mm_P5.00mm"
 		(layer "F.Cu")
-		(at 118.5 88 90)
+		(at 125.5 88 90)
 		(descr "C, Disc series, Radial, pin pitch=5.00mm, , diameter*width=7*2.5mm^2, Capacitor, http://cdn-reichelt.de/documents/datenblatt/B300/DS_KERKO_TC.pdf")
 		(tags "C Disc series Radial pin pitch 5.00mm  diameter 7mm width 2.5mm Capacitor")
@@
 	(footprint "Resistor_THT:R_Axial_DIN0204_L3.6mm_D1.6mm_P7.62mm_Horizontal"
 		(layer "F.Cu")
-		(at 113 82 -90)
+		(at 120 82 -90)
 		(descr "Resistor, Axial_DIN0204 series, Axial, Horizontal, pin pitch=7.62mm, 0.167W, length*diameter=3.6*1.6mm^2, http://cdn-reichelt.de/documents/datenblatt/B400/1_4W%23YAG.pdf")
 		(tags "Resistor Axial_DIN0204 series Axial Horizontal pin pitch 7.62mm 0.167W length 3.6mm diameter 1.6mm")
@@
 	(footprint "Capacitor_THT:C_Disc_D7.0mm_W2.5mm_P5.00mm"
 		(layer "F.Cu")
-		(at 120 60.5 -90)
+		(at 111 60.5 -90)
 		(descr "C, Disc series, Radial, pin pitch=5.00mm, , diameter*width=7*2.5mm^2, Capacitor, http://cdn-reichelt.de/documents/datenblatt/B300/DS_KERKO_TC.pdf")
 		(tags "C Disc series Radial pin pitch 5.00mm  diameter 7mm width 2.5mm Capacitor")
@@
 	)
 	(segment
-		(start 144.85 84.69)
-		(end 139.37 79.21)
+		(start 117.25 66.75)
+		(end 111 60.5)
 		(width 0.5)
 		(layer "B.Cu")
@@
 	)
 	(segment
-		(start 153.5 73.934874)
-		(end 153.5 59.04)
-		(width 0.5)
-		(layer "B.Cu")
-		(net 3)
-	)
-	(segment
-		(start 126.25 66.75)
-		(end 135.87 66.75)
-		(width 0.5)
-		(layer "B.Cu")
-		(net 3)
-	)
-	(segment
-		(start 156.5 84.69)
-		(end 144.85 84.69)
+		(start 138.58 80.92)
+		(end 135.58 80.92)
 		(width 0.5)
 		(layer "B.Cu")
@@
 	)
 	(segment
-		(start 136.08 73.5)
-		(end 139 73.5)
+		(start 153.5 73.934874)
+		(end 153.5 59.04)
 		(width 0.5)
 		(layer "B.Cu")
@@
 	)
 	(segment
-		(start 137.66 80.92)
-		(end 135.58 80.92)
+		(start 111.5 55.5)
+		(end 111 56)
 		(width 0.5)
 		(layer "B.Cu")
@@
 	)
 	(segment
-		(start 138.244214 77.63)
-		(end 139.37 78.755786)
+		(start 140 79.5)
+		(end 138.58 80.92)
 		(width 0.5)
 		(layer "B.Cu")
@@
 	)
 	(segment
-		(start 111.5 55)
-		(end 117 60.5)
+		(start 105 66.5)
+		(end 105 84)
 		(width 0.5)
 		(layer "B.Cu")
@@
 	)
 	(segment
-		(start 135.08 81.42)
-		(end 135.08 83.5)
-		(width 0.5)
-		(layer "B.Cu")
-		(net 3)
-	)
-	(segment
-		(start 137.62 68.5)
-		(end 136.08 70.04)
+		(start 111.5 55)
+		(end 111.5 55.5)
 		(width 0.5)
 		(layer "B.Cu")
@@
 	)
 	(segment
-		(start 139.37 79.21)
-		(end 137.66 80.92)
+		(start 135.58 80.92)
+		(end 135.08 81.42)
 		(width 0.5)
 		(layer "B.Cu")
@@
 	)
 	(segment
-		(start 157 77.434874)
-		(end 153.5 73.934874)
+		(start 136.08 70.04)
+		(end 137.62 68.5)
 		(width 0.5)
 		(layer "B.Cu")
@@
 	)
 	(segment
-		(start 140 74.5)
-		(end 140 77)
+		(start 135.87 66.75)
+		(end 117.25 66.75)
 		(width 0.5)
 		(layer "B.Cu")
@@
 	)
 	(segment
-		(start 139.37 77.63)
-		(end 138.244214 77.63)
+		(start 135.08 81.42)
+		(end 135.08 83.5)
 		(width 0.5)
 		(layer "B.Cu")
@@
 	)
 	(segment
-		(start 120 60.5)
-		(end 126.25 66.75)
+		(start 157 77.434874)
+		(end 153.5 73.934874)
 		(width 0.5)
 		(layer "B.Cu")
@@
 	)
 	(segment
-		(start 105 88.5)
-		(end 105 78)
+		(start 136.08 72.08)
+		(end 136.08 70.04)
 		(width 0.5)
 		(layer "B.Cu")
@@
 	)
 	(segment
-		(start 135.87 66.75)
-		(end 137.62 68.5)
+		(start 156.5 84.69)
+		(end 145.19 84.69)
 		(width 0.5)
 		(layer "B.Cu")
@@
 	)
 	(segment
-		(start 136.08 70.04)
-		(end 136.08 73.5)
+		(start 140 74.5)
+		(end 139 73.5)
 		(width 0.5)
 		(layer "B.Cu")
@@
 	)
 	(segment
-		(start 120 60.5)
-		(end 120 60)
+		(start 111 56)
+		(end 111 60.5)
 		(width 0.5)
 		(layer "B.Cu")
@@
 	)
 	(segment
-		(start 135.58 80.92)
-		(end 135.08 81.42)
+		(start 139 73.5)
+		(end 137.5 73.5)
 		(width 0.5)
 		(layer "B.Cu")
@@
 	)
 	(segment
-		(start 105 78)
-		(end 105 75.5)
+		(start 137.62 68.5)
+		(end 135.87 66.75)
 		(width 0.5)
 		(layer "B.Cu")
@@
 	)
 	(segment
-		(start 139 73.5)
-		(end 140 74.5)
+		(start 137.5 73.5)
+		(end 136.08 72.08)
 		(width 0.5)
 		(layer "B.Cu")
@@
 	)
 	(segment
-		(start 138.1 97.46)
-		(end 136.25 95.61)
+		(start 111 60.5)
+		(end 105 66.5)
 		(width 0.5)
 		(layer "B.Cu")
@@
 	)
 	(segment
-		(start 157 84.19)
-		(end 157 77.434874)
+		(start 105 84)
+		(end 105 88.5)
 		(width 0.5)
 		(layer "B.Cu")
@@
 	)
 	(segment
-		(start 105 75.5)
-		(end 120 60.5)
+		(start 140 79.5)
+		(end 140 74.5)
 		(width 0.5)
 		(layer "B.Cu")
@@
 	)
 	(segment
-		(start 140 77)
-		(end 139.37 77.63)
+		(start 138.1 97.46)
+		(end 136.25 95.61)
 		(width 0.5)
 		(layer "B.Cu")
@@
 	)
 	(segment
-		(start 117 60.5)
-		(end 120 60.5)
+		(start 145.19 84.69)
+		(end 140 79.5)
 		(width 0.5)
 		(layer "B.Cu")
@@
 	)
 	(segment
-		(start 139.37 78.755786)
-		(end 139.37 79.21)
+		(start 157 84.19)
+		(end 157 77.434874)
 		(width 0.5)
 		(layer "B.Cu")
@@
 	)
 	(segment
-		(start 113 89.62)
-		(end 116.88 89.62)
+		(start 123.88 89.62)
+		(end 120 89.62)
 		(width 0.5)
 		(layer "B.Cu")
@@
 	)
 	(segment
-		(start 116.88 89.62)
-		(end 118.5 88)
+		(start 125.5 88)
+		(end 123.88 89.62)
 		(width 0.5)
 		(layer "B.Cu")
@@
 	)
 	(segment
-		(start 118.5 88)
+		(start 125.5 88)
 		(end 132 88)
 		(width 0.5)
@@
 	)
 	(segment
-		(start 128.25 83)
-		(end 128.25 82.775126)
-		(width 0.5)
-		(layer "B.Cu")
-		(net 18)
-	)
-	(segment
-		(start 137.245786 79.92)
-		(end 138.182893 78.982893)
-		(width 0.5)
-		(layer "B.Cu")
-		(net 18)
-	)
-	(segment
-		(start 133.585786 81.5)
-		(end 135.165786 79.92)
-		(width 0.5)
-		(layer "B.Cu")
-		(net 18)
-	)
-	(segment
-		(start 135.08 68.5)
-		(end 135.08 75.88)
-		(width 0.5)
-		(layer "B.Cu")
-		(net 18)
-	)
-	(segment
-		(start 118.5 83)
-		(end 128.25 83)
-		(width 0.5)
-		(layer "B.Cu")
-		(net 18)
-	)
-	(segment
-		(start 128.25 82.775126)
-		(end 129.525126 81.5)
+		(start 135.87 76.67)
+		(end 135.87 78.13)
 		(width 0.5)
 		(layer "B.Cu")
@@
 	)
 	(segment
-		(start 129.525126 81.5)
-		(end 133.585786 81.5)
+		(start 135.87 78.13)
+		(end 134.5 79.5)
 		(width 0.5)
 		(layer "B.Cu")
@@
 	)
 	(segment
-		(start 138.182893 78.982893)
-		(end 136.83 77.63)
+		(start 135.08 75.88)
+		(end 135.87 76.67)
 		(width 0.5)
 		(layer "B.Cu")
@@
 	)
 	(segment
-		(start 135.87 77.63)
-		(end 135.87 76.67)
+		(start 125 83)
+		(end 124 82)
 		(width 0.5)
 		(layer "B.Cu")
@@
 	)
 	(segment
-		(start 135.87 76.67)
+		(start 135.08 68.5)
 		(end 135.08 75.88)
 		(width 0.5)
@@
 	)
 	(segment
-		(start 114 83)
-		(end 118.5 83)
+		(start 129 79.5)
+		(end 125.5 83)
 		(width 0.5)
 		(layer "B.Cu")
@@
 	)
 	(segment
-		(start 113 82)
-		(end 114 83)
+		(start 125.5 83)
+		(end 125 83)
 		(width 0.5)
 		(layer "B.Cu")
@@
 	)
 	(segment
-		(start 136.83 77.63)
-		(end 135.87 77.63)
+		(start 134.5 79.5)
+		(end 129 79.5)
 		(width 0.5)
 		(layer "B.Cu")
@@
 	)
 	(segment
-		(start 135.165786 79.92)
-		(end 137.245786 79.92)
+		(start 124 82)
+		(end 120 82)
 		(width 0.5)
 		(layer "B.Cu")
@@
 	)
 	(segment
-		(start 107.5 78)
-		(end 111.5 78)
+		(start 111.5 78)
+		(end 107.5 82)
+		(width 0.5)
+		(layer "B.Cu")
+		(net 23)
+	)
+	(segment
+		(start 107.5 82)
+		(end 107.5 84)
 		(width 0.5)
 		(layer "B.Cu")

Commit message: soucis_drill_invisible_rectifié
Other:
- board text added: "Yanis et Tristan"
Changed lines of the file:
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@@
 			(outputformat 4)
 			(mirror no)
-			(drillshape 0)
+			(drillshape 2)
 			(scaleselection 1)
 			(outputdirectory "../Gerber/")
@@
 		(layer "Edge.Cuts")
 	)
+	(gr_text "Yanis et Tristan"
+		(at 163.5 85.5 -90)
+		(layer "B.Cu")
+		(effects
+			(font
+				(size 1.5 1.5)
+				(thickness 0.3)
+				(bold yes)
+			)
+			(justify left bottom mirror)
+		)
+	)
 	(segment

Commit message: soft_ware_beginning
Parts:
- C1: value C -> 1pf
- C2, C3: value C -> 100nf
- C4: value C -> 0.1µf
- C5: value C -> 100n
- R1: value R -> 10k
- R2, R3: value R -> 100k
- R4: value R -> 1k
- R5: value R -> 47k
Changed lines of the file:
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@@
 			)
 		)
-		(property "Value" "C"
+		(property "Value" "0.1µf"
 			(at 2.5 2.5 90)
 			(layer "F.Fab")
@@
 		(tags "C Disc series Radial pin pitch 5.00mm  diameter 7mm width 2.5mm Capacitor")
 		(property "Reference" "C5"
-			(at 0 -3.5 90)
+			(at 2.5 -2.5 90)
 			(layer "F.SilkS")
 			(effects
@@
 			)
 		)
-		(property "Value" "C"
+		(property "Value" "100n"
 			(at 2.5 2.5 90)
 			(layer "F.Fab")
@@
 			)
 		)
-		(property "Value" "R"
+		(property "Value" "100k"
 			(at 3.81 1.92 90)
 			(layer "F.Fab")
@@
 			)
 		)
-		(property "Value" "C"
+		(property "Value" "100nf"
 			(at 2.5 2.5 0)
 			(layer "F.Fab")
@@
 			(at 2.5 -2.5 90)
 			(layer "F.SilkS")
+			(hide yes)
 			(effects
 				(font
@@
 			)
 		)
-		(property "Value" "C"
+		(property "Value" "1pf"
 			(at 2.5 2.5 90)
 			(layer "F.Fab")
@@
 			)
 		)
-		(property "Value" "R"
+		(property "Value" "1k"
 			(at 3.81 1.92 0)
 			(layer "F.Fab")
@@
 			)
 		)
-		(property "Value" "R"
+		(property "Value" "47k"
 			(at 3.81 1.92 90)
 			(layer "F.Fab")
@@
 			)
 		)
-		(property "Value" "R"
+		(property "Value" "100k"
 			(at 3.81 1.92 90)
 			(layer "F.Fab")
@@
 			)
 		)
-		(property "Value" "R"
+		(property "Value" "10k"
 			(at 3.81 1.92 0)
 			(layer "F.Fab")
@@
 			)
 		)
-		(property "Value" "C"
+		(property "Value" "100nf"
 			(at 2.5 2.5 90)
 			(layer "F.Fab")
